File: gaia-LTE/gaia-4gmodul.kicad_pcb (KiCad board)
At the start: 4 copper layers, 50 x 50 mm, 24 parts, among them J1 4G antenna connector(U.FL), J6 Global Connector Technology S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, Q1 DTC143ZEBTL, Q3 DTC143ZEBTL, Q4 DTC143ZEBTL, U1 SIM7600E-H, U2 Gaia Connector A, U3 Gaia Connector B

Commit message: ready
Connections:
- U1 pad 59: unconnected-(U1-AUX_ANT-Pad59) -> Net-(U1-AUX_ANT)
Changed lines of the file:
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@@
 	(net 22 "unconnected-(U1-SD_DATA0-Pad22)")
 	(net 23 "unconnected-(U1-RXD-Pad68)")
-	(net 24 "unconnected-(U1-AUX_ANT-Pad59)")
+	(net 24 "Net-(U1-AUX_ANT)")
 	(net 25 "unconnected-(U1-SD_DATA3-Pad25)")
 	(net 26 "unconnected-(U1-GNSS_ANT-Pad79)")
@@
 			(size 1.8 0.6)
 			(layers "F.Cu" "F.Mask" "F.Paste")
-			(net 24 "unconnected-(U1-AUX_ANT-Pad59)")
+			(net 24 "Net-(U1-AUX_ANT)")
 			(pinfunction "AUX_ANT")
-			(pintype "input+no_connect")
-			(solder_mask_margin 0.102)
-		)
+			(pintype "input")
+			(solder_mask_margin 0.102)
+		)

Commit message: USB fix
Connections:
- U1 pad 59: Net-(U1-AUX_ANT) -> unconnected-(U1-AUX_ANT-Pad59)
- U3 pad 15: unconnected-(U3-NC-Pad15) -> /USB_DN
- U3 pad 16: unconnected-(U3-NC-Pad16) -> /USB_DP
Routing:
- net /USB_DN: track 0.00 -> 9.69 mm
- net /USB_DP: track 0.00 -> 4.69 mm
Changed lines of the file:
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@@
 	(net 22 "unconnected-(U1-SD_DATA0-Pad22)")
 	(net 23 "unconnected-(U1-RXD-Pad68)")
-	(net 24 "Net-(U1-AUX_ANT)")
+	(net 24 "unconnected-(U1-AUX_ANT-Pad59)")
 	(net 25 "unconnected-(U1-SD_DATA3-Pad25)")
 	(net 26 "unconnected-(U1-GNSS_ANT-Pad79)")
@@
 	(net 87 "/VOUT_B2")
 	(net 88 "-BATT")
-	(net 89 "unconnected-(U3-NC-Pad15)")
-	(net 90 "unconnected-(U3-NC-Pad16)")
-	(net 91 "unconnected-(U1-USIM_DET-Pad53)")
-	(net 92 "unconnected-(J6-VPP-Pad6)")
-	(net 93 "unconnected-(U1-COEX3-Pad86)")
-	(net 94 "unconnected-(U1-COEX2-Pad84)")
+	(net 89 "unconnected-(U1-USIM_DET-Pad53)")
+	(net 90 "unconnected-(J6-VPP-Pad6)")
+	(net 91 "unconnected-(U1-COEX3-Pad86)")
+	(net 92 "unconnected-(U1-COEX2-Pad84)")
 	(footprint "Resistor_SMD:R_0402_1005Metric"
 		(layer "F.Cu")
@@
 			(size 1.8 0.6)
 			(layers "F.Cu" "F.Mask" "F.Paste")
-			(net 91 "unconnected-(U1-USIM_DET-Pad53)")
+			(net 89 "unconnected-(U1-USIM_DET-Pad53)")
 			(pinfunction "USIM_DET")
 			(pintype "bidirectional+no_connect")
@@
 			(size 1.8 0.6)
 			(layers "F.Cu" "F.Mask" "F.Paste")
-			(net 24 "Net-(U1-AUX_ANT)")
+			(net 24 "unconnected-(U1-AUX_ANT-Pad59)")
 			(pinfunction "AUX_ANT")
-			(pintype "input")
+			(pintype "input+no_connect")
 			(solder_mask_margin 0.102)
 		)
@@
 			(size 0.6 1.8)
 			(layers "F.Cu" "F.Mask" "F.Paste")
-			(net 94 "unconnected-(U1-COEX2-Pad84)")
+			(net 92 "unconnected-(U1-COEX2-Pad84)")
 			(pinfunction "COEX2")
 			(pintype "bidirectional+no_connect")
@@
 			(size 0.6 1.8)
 			(layers "F.Cu" "F.Mask" "F.Paste")
-			(net 93 "unconnected-(U1-COEX3-Pad86)")
+			(net 91 "unconnected-(U1-COEX3-Pad86)")
 			(pinfunction "COEX3")
 			(pintype "bidirectional+no_connect")
@@
 			(layers "*.Cu" "*.Mask")
 			(remove_unused_layers no)
-			(net 89 "unconnected-(U3-NC-Pad15)")
+			(net 43 "/USB_DN")
 			(pinfunction "NC")
-			(pintype "no_connect")
+			(pintype "unspecified")
 		)
 		(pad "16" thru_hole rect
@@
 			(layers "*.Cu" "*.Mask")
 			(remove_unused_layers no)
-			(net 90 "unconnected-(U3-NC-Pad16)")
+			(net 34 "/USB_DP")
 			(pinfunction "NC")
-			(pintype "no_connect")
+			(pintype "unspecified")
 		)
 		(pad "17" thru_hole rect
@@
 			(net 72 "unconnected-(U2-NC-Pad11)")
 			(pinfunction "NC")
-			(pintype "no_connect")
+			(pintype "unspecified")
 		)
 		(pad "12" thru_hole rect
@@
 			(net 73 "unconnected-(U2-NC-Pad12)")
 			(pinfunction "NC")
-			(pintype "no_connect")
+			(pintype "unspecified")
 		)
 		(pad "13" thru_hole rect
@@
 			(layers "B.Cu" "B.Mask" "B.Paste")
 			(roundrect_rratio 0.25)
-			(net 92 "unconnected-(J6-VPP-Pad6)")
+			(net 90 "unconnected-(J6-VPP-Pad6)")
 			(pinfunction "VPP")
 			(pintype "input+no_connect")
@@
 	)
 	(segment
+		(start 171.876938 96.5)
+		(end 171.086938 96.5)
+		(width 0.4)
+		(layer "F.Cu")
+		(net 34)
+	)
+	(segment
+		(start 172.777938 95.599)
+		(end 171.876938 96.5)
+		(width 0.4)
+		(layer "F.Cu")
+		(net 34)
+	)
+	(segment
+		(start 174.096938 94)
+		(end 173.269938 94)
+		(width 0.4)
+		(layer "F.Cu")
+		(net 34)
+	)
+	(segment
+		(start 172.777938 94.492)
+		(end 172.777938 95.599)
+		(width 0.4)
+		(layer "F.Cu")
+		(net 34)
+	)
+	(segment
+		(start 173.269938 94)
+		(end 172.777938 94.492)
+		(width 0.4)
+		(layer "F.Cu")
+		(net 34)
+	)
+	(segment
+		(start 172.767938 93.456)
+		(end 169.104938 93.456)
+		(width 0.4)
+		(layer "F.Cu")
+		(net 43)
+	)
+	(segment
+		(start 168.951938 93.609)
+		(end 168.951938 95.417)
+		(width 0.4)
+		(layer "F.Cu")
+		(net 43)
+	)
+	(segment
+		(start 173.223938 93)
+		(end 172.767938 93.456)
+		(width 0.4)
+		(layer "F.Cu")
+		(net 43)
+	)
+	(segment
+		(start 168.951938 95.417)
+		(end 167.868938 96.5)
+		(width 0.4)
+		(layer "F.Cu")
+		(net 43)
+	)
+	(segment
+		(start 169.104938 93.456)
+		(end 168.951938 93.609)
+		(width 0.4)
+		(layer "F.Cu")
+		(net 43)
+	)
+	(segment
+		(start 167.868938 96.5)
+		(end 166.916938 96.5)
+		(width 0.4)
+		(layer "F.Cu")
+		(net 43)
+	)
+	(segment
+		(start 174.096938 93)
+		(end 173.223938 93)
+		(width 0.4)
+		(layer "F.Cu")
+		(net 43)
+	)
+	(segment

Commit message: -
Parts:
- removed the C3 at (177.5, 99.5)
- removed J6: Global Connector Technology SIM8060-6-0-14-00-A, Connector_Card:nanoSIM_GCT_SIM8060-6-0-14-00
- removed R20: 0, Resistor_SMD:R_0603_1608Metric
- added C10: 100nF, Capacitor_SMD:C_0603_1608Metric, B.Cu at (188.5, 67.6)
- added C11: 4.7uF, Capacitor_SMD:C_0603_1608Metric, F.Cu at (177.7, 114.4)
- added C12: 100nF, Capacitor_SMD:C_0402_1005Metric, F.Cu at (176.5, 114.4)
- added C13: 1uF, Capacitor_SMD:C_0805_2012Metric, F.Cu at (179.5, 114.4)
- added C14: 1uF, Capacitor_SMD:C_0805_2012Metric, F.Cu at (190.4, 112.3)
- added C15: 100nF, Capacitor_SMD:C_0603_1608Metric, F.Cu at (171.9, 78.4)
- added J3: Micro_SD_Card_Det2, Connector_Card:microSD_HC_Hirose_DM3D-SF, B.Cu at (182.3, 106.3)
- added J4: SIM8051-6-0-14-00-A_REVD6, gaia-4gmodul-footprints:GCT_SIM8051-6-0-14-00-A_REVD6, B.Cu at (181.0, 73.5)
- added Q4: DTC143ZEBTL, gaia-4gmodul-footprints:DTC143ZEBTL, F.Cu at (171.9, 76.5)
- added U4: ADP3338AKCZ-2.85R7, gaia-4gmodul-footprints:ADP3338AKCZ-2.85R7, F.Cu at (184.9, 112.3)
- U1: renamed from U2; footprint gaia-4gmodul-footprints:Gaia_connector_4_6layer -> gaia-4gmodul-footprints:Gaia_connector_2_4layer
- U2: renamed from U3; footprint gaia-4gmodul-footprints:Gaia_connector_4_6layer -> gaia-4gmodul-footprints:Gaia_connector_2_4layer
- moved C1 1.66 mm to (168.2, 78.5)
- moved Q3 1.66 mm to (168.2, 76.6)
- renumbered C47 to C1, C4 to C3, C18 to C4, C51 to C5, C24 to C6, C20 to C7, C50 to C8, C49 to C9, D2 to D1, D1 to D2, Q4 to Q1, Q1 to Q2, R12 to R1, R13 to R2, R19 to R4, U1 to U3
Connections:
- C2 pad 1: /VOUT_B2 -> Vbat
- C3 pad 1: /VOUT_B2 -> Vbat
- C4 pad 1: /VOUT_B2 -> Vbat
- C5 pad 1: /VOUT_B2 -> Vbat
- C6 pad 1: /VOUT_B2 -> Vbat
- C7 pad 1: /VOUT_B2 -> Vbat
- D1 pad 2: /VOUT_B2 -> Vbat
- D2 pad 2: /VOUT_B2 -> Vbat
- U1 pad 1: /VOUT_A1 -> unconnected-(U1-VOUT_A1-Pad1)
- U1 pad 10: /VOUT_B2 -> unconnected-(U1-VOUT_B2-Pad10)
- U1 pad 11: unconnected-(U2-NC-Pad11) -> /pwrkey_input
- U1 pad 12: unconnected-(U2-NC-Pad12) -> /reset_input
- U1 pad 17: +BATT -> unconnected-(U1-+BATT-Pad17)
- U1 pad 18: +BATT -> unconnected-(U1-+BATT-Pad18)
- U1 pad 19: -BATT -> unconnected-(U1--BATT-Pad19)
- U1 pad 2: /VOUT_A1 -> unconnected-(U1-VOUT_A1-Pad2)
- U1 pad 20: -BATT -> unconnected-(U1--BATT-Pad20)
- U1 pad 3: /VOUT_A2 -> Vbat
- U1 pad 4: /VOUT_A2 -> unconnected-(U1-VOUT_A2-Pad4)
- U1 pad 5: /VOUT_A3 -> unconnected-(U1-VOUT_A3-Pad5)
- U1 pad 6: /VOUT_A3 -> unconnected-(U1-VOUT_A3-Pad6)
- U1 pad 7: /VOUT_B1 -> unconnected-(U1-VOUT_B1-Pad7)
- U1 pad 8: /VOUT_B1 -> unconnected-(U1-VOUT_B1-Pad8)
- U1 pad 9: /VOUT_B2 -> unconnected-(U1-VOUT_B2-Pad9)
- U2 pad 1: I2C_1_SDA -> unconnected-(U2-I2C_1_SCL-Pad1)
- U2 pad 11: /EXP0_USART_TXD -> unconnected-(U2-EXP2_USART_TXD-Pad11)
- U2 pad 12: /EXP2_USART_TXD -> unconnected-(U2-EXP2_USART_TXD-Pad12)
- U2 pad 13: /EXP0_USART_RXD -> unconnected-(U2-EXP2_USART_RXD-Pad13)
- U2 pad 14: /EXP2_USART_RXD -> unconnected-(U2-EXP2_USART_RXD-Pad14)
- U2 pad 2: I2C_2_SDA -> unconnected-(U2-I2C_2_SDA-Pad2)
- U2 pad 3: I2C_1_SCL -> unconnected-(U2-I2C_1_SCL-Pad3)
- U2 pad 4: I2C_2_SCL -> unconnected-(U2-I2C_2_SCL-Pad4)
- U2 pad 5: SPI_0_MISO -> unconnected-(U2-SPI_0_MISO-Pad5)
- U2 pad 6: /EXP1_SPI_CS -> unconnected-(U2-EXP1_SPI_CS-Pad6)
- U2 pad 7: SPI_0_MOSI -> unconnected-(U2-SPI_0_MOSI-Pad7)
- U2 pad 9: SPI_0_SCLK -> unconnected-(U2-SPI_0_SCLK-Pad9)
- U3 pad 11: /VOUT_B2 -> Vbat
- U3 pad 21: unconnected-(U1-SD_CMD-Pad21) -> /SD_CMD
- U3 pad 22: unconnected-(U1-SD_DATA0-Pad22) -> /SD_DAT0
- U3 pad 23: unconnected-(U1-SD_DATA1-Pad23) -> /SD_DAT1
- U3 pad 24: unconnected-(U1-SD_DATA2-Pad24) -> /SD_DAT2
- U3 pad 25: unconnected-(U1-SD_DATA3-Pad25) -> /SD_DAT3
- U3 pad 26: unconnected-(U1-SD_CLK-Pad26) -> /SD_CLK
- U3 pad 3: Net-(U1-PWRKEY) -> /pwrkey
- U3 pad 38: /VOUT_B2 -> Vbat
- U3 pad 39: /VOUT_B2 -> Vbat
- U3 pad 62: /VOUT_B2 -> Vbat
- U3 pad 63: /VOUT_B2 -> Vbat
Routing:
- net /VOUT_B2: track 87.8 -> 0.00 mm, vias 9 -> 0
- net GND: track 117.2 -> 48.8 mm, vias 28 -> 46
- net /reset_input: track 0.00 -> 53.3 mm, vias 0 -> 3
- net Vbat: track 0.00 -> 48.7 mm, vias 0 -> 11
- net /pwrkey_input: track 0.00 -> 43.6 mm, vias 0 -> 3
- net /USIM_VDD: track 5.93 -> 46.1 mm
- net /USIM_RESET: track 6.47 -> 35.7 mm, vias 1 -> 2
- net /USIM_CLK: track 10.0 -> 36.5 mm, vias 1 -> 2
- net /USB_DP: track 4.69 -> 27.6 mm, vias 0 -> 1
- net /USB_DN: track 9.69 -> 27.7 mm, vias 0 -> 1
- net /sdCard/SD_2.85V: track 0.00 -> 14.4 mm, vias 0 -> 1
- net /USIM_DATA: track 10.9 -> 21.6 mm, vias 1 -> 2
- net /pwrkey: track 0.00 -> 9.81 mm, vias 0 -> 2
- net /SD_DAT0: track 0.00 -> 8.52 mm, vias 0 -> 1
- net /SD_DAT1: track 0.00 -> 8.50 mm, vias 0 -> 1
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- added copper zone on In4.Cu, net GND
- added copper zone on In2.Cu, net Vbat
- removed copper zone on In2.Cu, net /VOUT_B2
Other:
- copper layers 4 -> 6
