File: gaia-LTE/sdcardpsu.kicad_sch (KiCad schematic)
At the start: 3 parts, among them U4 ADP3338AKCZ-2.85R7

Commit message: preparing to install TVS
Parts:
- removed C13, C14: 1uF, Capacitor_SMD:C_0805_2012Metric, symbol Device:C_Small
- removed U4: ADP3338AKCZ-2.85R7, gaia-4gmodul-footprints:ADP3338AKCZ-2.85R7, symbol gaia-4gmodul-symbols:ADP3338AKCZ-2.85R7
Connections:
- no-connect marks 1 -> 0
