File: gaia-lte.kicad_pcb (KiCad board)
At the start: 6 copper layers, 50 x 50 mm, 31 parts, among them J1 4G antenna connector(U.FL), J3 Micro_SD_Card_Det2, J4 SIM8051-6-0-14-00-A_REVD6, Q1 DTC143ZEBTL, Q2 DTC143ZEBTL, Q3 DTC143ZEBTL, Q4 DTC143ZEBTL, U1 Gaia Connector A, U2 Gaia Connector B, U3 SIM7600E-H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

Commit message: ready for production
Parts:
- removed J3: Micro_SD_Card_Det2, Connector_Card:microSD_HC_Hirose_DM3D-SF
- removed U2: Gaia Connector B, gaia-4gmodul-footprints:Gaia_connector_2_4layer
- removed U4: ADP3338AKCZ-2.85R7, gaia-4gmodul-footprints:ADP3338AKCZ-2.85R7
- added C16: NM_NC, Capacitor_SMD:C_0402_1005Metric, F.Cu at (205.7, 78.0)
- added C17: NM_NC, Capacitor_SMD:C_0402_1005Metric, F.Cu at (205.7, 75.2)
- added C18: 220uF, Capacitor_SMD:CP_Elec_5x5.9, B.Cu at (195.0, 88.5)
- added D10: ESD9M5, Diode_SMD:D_SOD-923, F.Cu at (183.6, 113.4)
- added D11: ESD9M5, Diode_SMD:D_SOD-923, F.Cu at (181.3, 113.4)
- added D12: ESD9M5, Diode_SMD:D_SOD-923, F.Cu at (180.2, 113.4)
- added D13: ESD9M5, Diode_SMD:D_SOD-923, F.Cu at (179.2, 113.4)
- added D14: ESD9M5, Diode_SMD:D_SOD-923, F.Cu at (182.4, 113.4)
- added D3: MMSZ5231BT1G, Diode_SMD:D_SOD-123, F.Cu at (193.8, 72.2)
- added D4: ESD9M5.0ST5G, Diode_SMD:D_SOD-923, F.Cu at (195.4, 73.9)
- added D5: ESD9M5, Diode_SMD:D_SOD-923, F.Cu at (186.8, 113.4)
- added D6: ESD9L5.0ST5G, Diode_SMD:D_SOD-923, B.Cu at (167.8, 102.5)
- added D7: ESD9L5.0ST5G, Diode_SMD:D_SOD-923, B.Cu at (170.2, 102.5)
- added D8: ESDA6V1W5, gaia-lte-footprints:SOT-23-5, F.Cu at (174.1, 71.2)
- added D9: ESD9M5, Diode_SMD:D_SOD-923, F.Cu at (185.7, 113.4)
- added J2: AUX Ant connector(u.fl), gaia-lte-footprints:U.FL_Hirose_U.FL-R-SMT-1_Vertical, F.Cu at (205.2, 72.6)
- added J5: SIM8051-6-0-14-00-A_REVD6, gaia-lte-footprints:GCT_SIM8051-6-0-14-00-A_REVD6, B.Cu at (181.0, 73.5)
- added J6: Conn_02x10_Odd_Even, gaia-lte-footprints:Gaia_connector_2_4layer, F.Cu at (169.0, 91.5)
- added J7: Conn_02x10_Odd_Even, gaia-lte-footprints:Gaia_connector_2_4layer, F.Cu at (209.4, 91.5)
- added R3: 0, Resistor_SMD:R_0402_1005Metric, F.Cu at (205.2, 76.6)
- added TP1: TestPoint, TestPoint:TestPoint_Pad_1.5x1.5mm, B.Cu at (204.3, 78.9)
- C10: value 100nF -> 1uF; footprint Capacitor_SMD:C_0603_1608Metric -> Capacitor_SMD:C_0402_1005Metric; moved to F.Cu
- C11: value 4.7uF -> 100nF; moved to B.Cu
- C13: footprint Capacitor_SMD:C_0805_2012Metric -> Capacitor_SMD:C_0402_1005Metric; moved to B.Cu
- C14: value 1uF -> 220uF; footprint Capacitor_SMD:C_0805_2012Metric -> Capacitor_SMD:CP_Elec_5x5.9; moved to B.Cu
- C2: value 220uF -> 1uF; footprint Capacitor_SMD:CP_Elec_5x5.9 -> Capacitor_SMD:C_0603_1608Metric; moved to F.Cu
- C3: value 220uF -> 1uF; footprint Capacitor_SMD:CP_Elec_5x5.9 -> Capacitor_SMD:C_0402_1005Metric; moved to F.Cu
- J1: footprint Connector_Coaxial:U.FL_Hirose_U.FL-R-SMT-1_Vertical -> gaia-lte-footprints:U.FL_Hirose_U.FL-R-SMT-1_Vertical
- J4: value SIM8051-6-0-14-00-A_REVD6 -> Micro_SD_Card_Det2; footprint gaia-4gmodul-footprints:GCT_SIM8051-6-0-14-00-A_REVD6 -> Connector_Card:microSD_HC_Hirose_DM3D-SF
- Q1, Q2, Q3, Q4: footprint gaia-4gmodul-footprints:DTC143ZEBTL -> gaia-lte-footprints:DTC143ZEBTL
- U1: value Gaia Connector A -> AP2127K-2.8; footprint gaia-4gmodul-footprints:Gaia_connector_2_4layer -> gaia-lte-footprints:SOT-23-5
- U3: footprint gaia-4gmodul-footprints:SIM7600 -> gaia-lte-footprints:SIM7600
- moved C10 48.6 mm to (175.6, 114.4), turned to -90 degrees
- moved C11 48.0 mm to (188.5, 67.6), turned to 180 degrees
- moved U1 40.6 mm to (173.7, 110.8), turned to -90 degrees
- moved C2 36.6 mm to (176.8, 114.3), turned to -90 degrees
- moved J4 32.9 mm to (182.3, 106.3), turned to 180 degrees
- moved C14 30.1 mm to (195.0, 82.5), turned to 180 degrees
- moved C3 28.7 mm to (174.2, 108.2)
- moved C13 23.3 mm to (174.9, 91.5), turned to 90 degrees
- moved C12 1.55 mm to (178.1, 114.4)
Connections:
- net /netlight renamed Net-(U3-NETLIGHT)
- net /pwrkey renamed Net-(U3-PWRKEY)
- net /reset renamed Net-(U3-RESET)
- net /status renamed Net-(U3-STATUS)
- C10 pad 1: GND -> +2V8
- C10 pad 2: /USIM_VDD -> GND
- C11 pad 1: /sdCard/SD_2.85V -> GND
- C11 pad 2: GND -> /USIM_VDD
- C12 pad 1: /sdCard/SD_2.85V -> +2V8
- C13 pad 1: /sdCard/SD_2.85V -> VBUS
- C14 pad 1: GND -> VBUS
- C14 pad 2: Vbat -> GND
- C2 pad 1: Vbat -> +2V8
- C3 pad 1: Vbat -> VBUS
- C4 pad 1: Vbat -> VBUS
- C5 pad 1: Vbat -> VBUS
- C6 pad 1: Vbat -> VBUS
- C7 pad 1: Vbat -> VBUS
- D1 pad 2: Vbat -> VBUS
- D2 pad 2: Vbat -> VBUS
- J4 pad 1: /USIM_VDD -> /SD_DAT2
- J4 pad 2: /USIM_RESET -> /SD_DAT3
- J4 pad 3: /USIM_CLK -> /SD_CMD
- J4 pad 4: GND -> +2V8
- J4 pad 5: GND -> /SD_CLK
- J4 pad 6: unconnected-(J4-VPP-Pad6) -> GND
- J4 pad 7: /USIM_DATA -> /SD_DAT0
- J4 pad 8: GND -> /SD_DAT1
- U1 pad 1: unconnected-(U1-VOUT_A1-Pad1) -> VBUS
- U1 pad 2: unconnected-(U1-VOUT_A1-Pad2) -> GND
- U1 pad 3: Vbat -> VBUS
- U1 pad 5: unconnected-(U1-VOUT_A3-Pad5) -> +2V8
- U3 pad 11: Vbat -> VBUS
- U3 pad 15: /VDD_1V8 -> unconnected-(U3-VDD_1V8-Pad15)
- U3 pad 38: Vbat -> VBUS
- U3 pad 39: Vbat -> VBUS
- U3 pad 59: unconnected-(U3-AUX_ANT-Pad59) -> Net-(U3-AUX_ANT)
- U3 pad 62: Vbat -> VBUS
- U3 pad 63: Vbat -> VBUS
- U3 pad 85: unconnected-(U3-BOOT_CFG0-Pad85) -> Net-(U3-BOOT_CFG0)
Routing:
- net VBUS: track 0.00 -> 51.0 mm, vias 0 -> 12
- net Vbat: track 48.7 -> 0.00 mm, vias 11 -> 0
- net /sdCard/SD_2.85V: track 14.4 -> 0.00 mm, vias 1 -> 0
- net +2V8: track 0.00 -> 12.3 mm, vias 0 -> 2
- net Net-(U3-AUX_ANT): track 0.00 -> 10.4 mm
- net /USIM_VDD: track 46.1 -> 56.2 mm, vias 1 -> 2
- net /USIM_DATA: track 21.6 -> 31.3 mm
- net GND: track 48.8 -> 57.8 mm, vias 46 -> 63
- net /USIM_RESET: track 35.7 -> 42.5 mm
- net /USIM_CLK: track 36.5 -> 43.1 mm
- net Net-(J2-In): track 0.00 -> 2.44 mm
- net Net-(U3-BOOT_CFG0): track 0.00 -> 2.09 mm, vias 0 -> 1
- net /SD_DAT1: track 8.50 -> 10.6 mm, vias 1 -> 2
- net /SD_DAT2: track 7.72 -> 9.04 mm
- net /SD_CLK: track 7.72 -> 9.04 mm
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- added copper zone on In2.Cu, net VBUS
- removed copper zone on In2.Cu, net Vbat
Other:
- board text added: "AUX"
- board text added: "GSM/LTE Module"
- board text added: "MAIN"
- board text added: "STAT"
- board text added: "revision 1.0"
- board text removed: "STATUS"
