File: gaia-lte.kicad_sch (KiCad schematic)
At the start: 54 parts, among them J1 4G antenna connector(U.FL), J2 AUX Ant connector(u.fl), J4 Micro_SD_Card_Det2, J5 SIM8051-6-0-14-00-A_REVD6, J6 Conn_02x10_Odd_Even, J7 Conn_02x10_Odd_Even, Q1 DTC143ZEBTL, Q2 DTC143ZEBTL, Q3 DTC143ZEBTL, Q4 DTC143ZEBTL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

Commit message: ready for production
Parts:
- removed R10, R11, R12: 22R, symbol Device:R_Small
- removed R8, R9: 0, Resistor_SMD:R_0402_1005Metric, symbol Device:R_Small
- C10, C13, C3: footprint Capacitor_SMD:C_1812_4532Metric -> Capacitor_SMD:C_0402_1005Metric
- C2: value 4.7uF -> 1uF
- D3: footprint (none) -> Diode_SMD:D_SOD-123
- D8, U1: footprint Package_TO_SOT_SMD:SOT-23-5 -> gaia-lte-footprints:SOT-23-5
- J1, J2: footprint Connector_Coaxial:U.FL_Hirose_U.FL-R-SMT-1_Vertical -> gaia-lte-footprints:U.FL_Hirose_U.FL-R-SMT-1_Vertical
- J5: footprint gaia-4gmodul-footprints:GCT_SIM8051-6-0-14-00-A_REVD6 -> gaia-lte-footprints:GCT_SIM8051-6-0-14-00-A_REVD6
- J6, J7: footprint gaia_obc-footprints:PinHeader_2x10_P2.00mm_Vertical_SMD -> gaia-lte-footprints:Gaia_connector_2_4layer
- Q1, Q2, Q3, Q4: footprint gaia-4gmodul-footprints:DTC143ZEBTL -> gaia-lte-footprints:DTC143ZEBTL
- U3: footprint gaia-4gmodul-footprints:SIM7600 -> gaia-lte-footprints:SIM7600
Connections:
- net GND: now also D6.2 (A2), J6.10 (Pin_10), J6.8 (Pin_8); no longer D6.1 (A1)
- net USB_DN: now also D6.1 (A1), U3.12 (USB_DN); no longer D6.2 (A2)
- net USB_DP: now also U3.13 (USB_DP)
- net USIM_CLK: now also J5.3 (CLK)
- net USIM_DATA: now also J5.7 (I/O)
- net USIM_RESET: now also J5.2 (RST)
- no-connect marks 45 -> 71

Commit message: header fix
Connections:
- net GND: now also J6.6 (Pin_6), J6.9 (Pin_9)
- no-connect marks 71 -> 69
Changed lines of the file:
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@@
 	)
 	(no_connect
-		(at 39.37 31.75)
-	)
-	(no_connect
 		(at 26.67 39.37)
 	)
@@
 	)
 	(no_connect
-		(at 26.67 36.83)
-	)
-	(no_connect
 		(at 153.67 74.93)
 	)
@@
 	(symbol
 		(lib_id "power:GND")
+		(at 39.37 31.75 90)
+		(unit 1)
+		(exclude_from_sim no)
+		(in_bom yes)
+		(on_board yes)
+		(dnp no)
+		(fields_autoplaced yes)
+		(property "Reference" "#PWR079"
+			(at 45.72 31.75 0)
+			(effects
+				(font
+					(size 1.27 1.27)
+				)
+				(hide yes)
+			)
+		)
+		(property "Value" "GND"
+			(at 43.18 31.7499 90)
+			(effects
+				(font
+					(size 1.27 1.27)
+				)
+				(justify right)
+			)
+		)
+		(property "Footprint" ""
+			(at 39.37 31.75 0)
+			(effects
+				(font
+					(size 1.27 1.27)
+				)
+				(hide yes)
+			)
+		)
+		(property "Datasheet" ""
+			(at 39.37 31.75 0)
+			(effects
+				(font
+					(size 1.27 1.27)
+				)
+				(hide yes)
+			)
+		)
+		(property "Description" "Power symbol creates a global label with name \"GND\" , ground"
+			(at 39.37 31.75 0)
+			(effects
+				(font
+					(size 1.27 1.27)
+				)
+				(hide yes)
+			)
+		)
+		(pin "1"
+		)
+		(instances
+			(project "gaia-lte"
+				(path "/7b77d13a-9a8b-42d2-a530-7929f32d7253"
+					(reference "#PWR079")
+					(unit 1)
+				)
+			)
+		)
+	)
+	(symbol
+		(lib_id "power:GND")
 		(at 222.25 85.09 90)
 		(unit 1)
@@
 					(unit 1)
 				)
+			)
+		)
+	)
+	(symbol
+		(lib_id "power:GND")
+		(at 26.67 36.83 270)
+		(unit 1)
+		(exclude_from_sim no)
+		(in_bom yes)
+		(on_board yes)
+		(dnp no)
+		(fields_autoplaced yes)
+		(property "Reference" "#PWR087"
+			(at 20.32 36.83 0)
+			(effects
+				(font
+					(size 1.27 1.27)
+				)
+				(hide yes)
+			)
+		)
+		(property "Value" "GND"
+			(at 22.86 36.8299 90)
+			(effects
+				(font
+					(size 1.27 1.27)
+				)
+				(justify right)
+			)
+		)
+		(property "Footprint" ""
+			(at 26.67 36.83 0)
+			(effects
+				(font
+					(size 1.27 1.27)
+				)
+				(hide yes)
+			)
+		)
+		(property "Datasheet" ""
+			(at 26.67 36.83 0)
+			(effects
+				(font
+					(size 1.27 1.27)
+				)
+				(hide yes)
+			)
+		)
+		(property "Description" "Power symbol creates a global label with name \"GND\" , ground"
+			(at 26.67 36.83 0)
+			(effects
+				(font
+					(size 1.27 1.27)
+				)
+				(hide yes)
+			)
+		)
+		(pin "1"
+		)
+		(instances
+			(project "gaia-lte"
+				(path "/7b77d13a-9a8b-42d2-a530-7929f32d7253"
+					(reference "#PWR087")
+					(unit 1)
+				)

Commit message: v1.1 - PROD
Parts:
- added R5, R6: 22, Resistor_SMD:R_0402_1005Metric, symbol Device:R_Small
Connections:
- net USB_DN: now also R5.1; no longer U3.12 (USB_DN)
- net USB_DP: now also R6.2; no longer U3.13 (USB_DP)
- new net: R5.2, U3.12 (USB_DN)
- new net: R6.1, U3.13 (USB_DP)
Changed lines of the file:
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@@
 	(wire
 		(pts
+			(xy 127 73.66) (xy 132.08 73.66)
+		)
+		(stroke
+			(width 0)
+			(type default)
+		)
+	)
+	(wire
+		(pts
 			(xy 207.01 26.67) (xy 207.01 24.13)
 		)
@@
 	(wire
 		(pts
-			(xy 110.49 76.2) (xy 134.62 76.2)
+			(xy 110.49 76.2) (xy 121.92 76.2)
 		)
 		(stroke
@@
 	(wire
 		(pts
-			(xy 116.84 73.66) (xy 132.08 73.66)
+			(xy 116.84 73.66) (xy 121.92 73.66)
 		)
 		(stroke
@@
 	(wire
 		(pts
+			(xy 127 76.2) (xy 134.62 76.2)
+		)
+		(stroke
+			(width 0)
+			(type default)
+		)
+	)
+	(wire
+		(pts
 			(xy 24.13 134.62) (xy 29.21 134.62)
 		)
@@
 	)
 	(symbol
+		(lib_id "Device:R_Small")
+		(at 124.46 73.66 90)
+		(mirror x)
+		(unit 1)
+		(exclude_from_sim no)
+		(in_bom yes)
+		(on_board yes)
+		(dnp no)
+		(property "Reference" "R5"
+			(at 124.46 68.58 90)
+			(effects
+				(font
+					(size 1.016 1.016)
+				)
+			)
+		)
+		(property "Value" "22"
+			(at 124.46 71.12 90)
+			(effects
+				(font
+					(size 1.27 1.27)
+				)
+			)
+		)
+		(property "Footprint" "Resistor_SMD:R_0402_1005Metric"
+			(at 124.46 73.66 0)
+			(effects
+				(font
+					(size 1.27 1.27)
+				)
+				(hide yes)
+			)
+		)
+		(property "Datasheet" "~"
+			(at 124.46 73.66 0)
+			(effects
+				(font
+					(size 1.27 1.27)
+				)
+				(hide yes)
+			)
+		)
+		(property "Description" "Resistor, small symbol"
+			(at 124.46 73.66 0)
+			(effects
+				(font
+					(size 1.27 1.27)
+				)
+				(hide yes)
+			)
+		)
+		(pin "2"
+		)
+		(pin "1"
+		)
+		(instances
+			(project "gaia-lte"
+				(path "/7b77d13a-9a8b-42d2-a530-7929f32d7253"
+					(reference "R5")
+					(unit 1)
+				)
+			)
+		)
+	)
+	(symbol
 		(lib_id "power:GND")
 		(at 80.01 137.16 0)
@@
 					(unit 1)
 				)
+			)
+		)
+	)
+	(symbol
+		(lib_id "Device:R_Small")
+		(at 124.46 76.2 270)
+		(mirror x)
+		(unit 1)
+		(exclude_from_sim no)
+		(in_bom yes)
+		(on_board yes)
+		(dnp no)
+		(property "Reference" "R6"
+			(at 124.46 81.28 90)
+			(effects
+				(font
+					(size 1.016 1.016)
+				)
+			)
+		)
+		(property "Value" "22"
+			(at 124.46 78.74 90)
+			(effects
+				(font
+					(size 1.27 1.27)
+				)
+			)
+		)
+		(property "Footprint" "Resistor_SMD:R_0402_1005Metric"
+			(at 124.46 76.2 0)
+			(effects
+				(font
+					(size 1.27 1.27)
+				)
+				(hide yes)
+			)
+		)
+		(property "Datasheet" "~"
+			(at 124.46 76.2 0)
+			(effects
+				(font
+					(size 1.27 1.27)
+				)
+				(hide yes)
+			)
+		)
+		(property "Description" "Resistor, small symbol"
+			(at 124.46 76.2 0)
+			(effects
+				(font
+					(size 1.27 1.27)
+				)
+				(hide yes)
+			)
+		)
+		(pin "2"
+		)
+		(pin "1"
+		)
+		(instances
+			(project "gaia-lte"
+				(path "/7b77d13a-9a8b-42d2-a530-7929f32d7253"
+					(reference "R6")
+					(unit 1)
+				)
